File: pcb_test/mod1.sch (KiCad schematic (older format))
At the start: 130 parts, among them J1 J1, J2 Screw_Terminal_01x03, J3 Screw_Terminal_01x03, J4 Screw_Terminal_01x03, J5 Screw_Terminal_01x03, K1 G6S-2, K2 G6S-2, Q1 SS8050, Q2 SS8050, Q3 MMBTA06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

Commit message: update on package module
Parts:
- R28: value 1% 390k -> 390k 1/10W; LCSC C17656 -> (none)
Changed lines of the file:
@@
 P 1800 7850
 F 0 "R28" H 1870 7896 50  0000 L CNN
-F 1 "1% 390k" H 1870 7805 50  0000 L CNN
+F 1 "390k 1/10W" H 1870 7805 50  0000 L CNN
 F 2 "Resistor_SMD:R_0603_1608Metric" V 1730 7850 50  0001 C CNN
 F 3 "~" H 1800 7850 50  0001 C CNN
-F 4 "C17656" H 1800 7850 50  0001 C CNN "LCSC"
 	1    1800 7850
 	1    0    0    -1
